Commit message: feat: 4-phase docking pipeline + sim
Signed-off-by: SHuttooo <matthieuvinet04@gmail.com>

File: ros2/src/openamrobot_description/urdf/gazebo_control.xacro (robot description, xacro)
@@ -1,5 +1,16 @@
 <?xml version="1.0"?>
 <robot xmlns:xacro="http://www.ros.org/wiki/xacro">
-  <!-- ── World-level plugins (no reference attribute) ─────────────── -->
+  <!--
+    World-level plugins.
+    DiffDrive: wheel_radius/wheel_separation must match the physical wheel
+    meshes. The upstream SolidWorks export had wheel_radius=0.11 in the plugin
+    but cylinder collisions of radius 0.10 on the wheel links; we keep them
+    in sync at 0.10 m. wheel_separation = 0.4075 m is the centre-to-centre
+    distance from the URDF wheel joint origins (±0.20375 m).
+    child_frame_id is base_footprint so the Gazebo-side odometry TF aligns
+    with the Nav2-convention TF chain produced by robot_state_publisher.
+    Topics are relative (no leading slash) so the plugin works correctly
+    when the robot is spawned inside a namespace.
+  -->
   <gazebo>
     <plugin filename="gz-sim-diff-drive-system" name="gz::sim::systems::DiffDrive">
@@ -7,5 +18,5 @@
       <right_joint>right_wheel_joint</right_joint>
       <wheel_separation>0.4075</wheel_separation>
-      <wheel_radius>0.11</wheel_radius>
+      <wheel_radius>0.1</wheel_radius>
       <max_linear_acceleration>0.5</max_linear_acceleration>
       <min_linear_acceleration>-0.5</min_linear_acceleration>
@@ -16,19 +27,19 @@
       <max_angular_velocity>2.0</max_angular_velocity>
       <min_angular_velocity>-2.0</min_angular_velocity>
-      <topic>/cmd_vel</topic>
+      <topic>cmd_vel</topic>
       <frame_id>odom</frame_id>
-      <child_frame_id>base_link</child_frame_id>
-      <odom_topic>/odom</odom_topic>
-      <tf_topic>/tf</tf_topic>
+      <child_frame_id>base_footprint</child_frame_id>
+      <odom_topic>odom</odom_topic>
+      <tf_topic>tf</tf_topic>
       <odom_publish_frequency>50</odom_publish_frequency>
     </plugin>
     <plugin filename="gz-sim-joint-state-publisher-system"
       name="gz::sim::systems::JointStatePublisher">
-      <topic>/joint_states</topic>
+      <topic>joint_states</topic>
       <joint_name>left_wheel_joint</joint_name>
       <joint_name>right_wheel_joint</joint_name>
     </plugin>
   </gazebo>
-  <!-- ── Link-level: base_link ─────────────────────────────────────── -->
+  <!-- base_link surface -->
   <gazebo reference="base_link">
     <material>Gazebo/White</material>
@@ -49,5 +60,5 @@
     </surface>
   </gazebo>
-  <!-- ── Link-level: left_wheel_link ────────────────────────────────────── -->
+  <!-- Drive wheels: high friction in rolling direction, low slip -->
   <gazebo reference="left_wheel_link">
     <material>Gazebo/DarkGrey</material>
@@ -72,5 +83,4 @@
     </surface>
   </gazebo>
-  <!-- ── Link-level: right_wheel_link ───────────────────────────────────── -->
   <gazebo reference="right_wheel_link">
     <material>Gazebo/DarkGrey</material>
@@ -95,6 +105,5 @@
     </surface>
   </gazebo>
-  <!-- ── Link-level: caster wheels ───────────────────────────────────── -->
-  <!-- We apply low friction to caster wheels to prevent them from catching and dragging in Gazebo -->
+  <!-- Casters: friction 0 so the drive wheels carry all the traction. -->
   <xacro:macro name="caster_gazebo" params="prefix">
     <gazebo reference="${prefix}_caster_link">
@@ -125,10 +134,15 @@
   <xacro:caster_gazebo prefix="bl" />
   <xacro:caster_gazebo prefix="br" />
-  <!-- ── Link-level: lidar_link — sensor ONLY here ─────────────────── -->
+  <!--
+    Lidar.
+    Range, samples and noise tuned for the docking simulation:
+      - 0.15 m near limit so the lidar can see close obstacles next to the robot
+      - 12 m far limit to span the 10x10 m room used by the docking scenario
+  -->
   <gazebo reference="lidar_link">
     <material>Gazebo/Black</material>
     <sensor name="lidar_sensor" type="gpu_lidar">
       <pose relative_to="lidar_link">0 0 0 0 0 0</pose>
-      <topic>/scan</topic>
+      <topic>scan</topic>
       <gz_frame_id>lidar_link</gz_frame_id>
       <update_rate>10</update_rate>
@@ -143,6 +157,6 @@
         </scan>
         <range>
-          <min>0.40</min>
-          <max>10.0</max>
+          <min>0.15</min>
+          <max>12.0</max>
           <resolution>0.01</resolution>
         </range>
@@ -157,3 +171,40 @@
     </sensor>
   </gazebo>
+  <!--
+    RGB camera.
+    640x480 @ 15 Hz is the maximum the gz<->ROS bridge handles reliably; HD
+    (1280x720) stalls the image bridge to ~0.2 Hz. horizontal_fov=1.2 rad
+    chosen to match the real-robot camera.
+    gz_frame_id is camera_rgb_optical_frame (declared in the main xacro) so
+    the image stream carries the -pi/2,-pi/2 rotation that apriltag_ros::solvePnP
+    expects when computing the tag pose.
+  -->
+  <gazebo reference="camera_link">
+    <material>Gazebo/Black</material>
+    <sensor name="rgb_camera" type="camera">
+      <pose relative_to="camera_link">0 0 0 0 0 0</pose>
+      <topic>camera/image_raw</topic>
+      <gz_frame_id>camera_rgb_optical_frame</gz_frame_id>
+      <update_rate>15</update_rate>
+      <camera>
+        <horizontal_fov>1.2</horizontal_fov>
+        <image>
+          <width>640</width>
+          <height>480</height>
+          <format>R8G8B8</format>
+        </image>
+        <clip>
+          <near>0.05</near>
+          <far>15.0</far>
+        </clip>
+        <noise>
+          <type>gaussian</type>
+          <mean>0.0</mean>
+          <stddev>0.005</stddev>
+        </noise>
+      </camera>
+      <always_on>true</always_on>
+      <visualize>false</visualize>
+    </sensor>
+  </gazebo>
 </robot>

File: ros2/src/openamrobot_description/urdf/robo_urdf.urdf.xacro (robot description, xacro)
@@ -1,9 +1,32 @@
 <?xml version="1.0" encoding="utf-8"?>
-<!-- This URDF was automatically created by SolidWorks to URDF Exporter! Originally created by
-Stephen Brawner (brawner@gmail.com)
-     Commit Version: 1.6.0-4-g7f85cfe  Build Version: 1.6.7995.38578
-     For more information, please see http://wiki.ros.org/sw_urdf_exporter -->
+<!--
+  OpenAMRobot differential-drive robot description.
+  Link/joint geometry and STL meshes originate from a SolidWorks-exported URDF
+  (sw_urdf_exporter, Stephen Brawner) by Niraj Dhakal (the upstream URDF author),
+  later packaged by Raj Indulkar in openamrobot-simulation. See top-level
+  NOTICE.md for the full attribution chain.
+  Modifications applied in this revision (openamrobot-docking contribution):
+    - added a base_footprint root link + base_joint (Nav2 TF convention)
+    - symmetrised left/right wheel inertials (off-diagonals set to 0 and the
+      two wheels made identical) — fixes the "robot circles when commanded
+      straight" failure caused by SolidWorks-exported asymmetries
+    - added camera_link and camera_rgb_optical_frame for AprilTag detection
+    - lidar range adjusted to 0.15-12 m (see gazebo_control.xacro)
+    - cylinder collisions on drive wheels with radius 0.10 m (reconciled
+      with the DiffDrive plugin wheel_radius — see gazebo_control.xacro)
+-->
 <robot
-  name="robo_urdf" xmlns:xacro="http://www.ros.org/wiki/xacro">
+  name="openamrobot" xmlns:xacro="http://www.ros.org/wiki/xacro">
+  <!--
+    base_footprint: ground-projection of base_link, Nav2 convention.
+    base_joint lifts base_link 0.053467 m so the drive-wheel centres sit at
+    z = wheel_radius = 0.10 m above the ground when base_footprint is at z=0.
+  -->
+  <link name="base_footprint"/>
+  <joint name="base_joint" type="fixed">
+    <origin xyz="0 0 0.053467" rpy="0 0 0"/>
+    <parent link="base_footprint"/>
+    <child link="base_link"/>
+  </joint>
   <link
     name="base_link">
@@ -466,19 +489,20 @@
     <dynamics damping="0.001" friction="0.001" />
   </joint>
+  <!--
+    Drive wheels.
+    Inertials made symmetric: off-diagonal terms zeroed and ixx = iyy = izz
+    forced to the same average so left and right behave identically. The
+    SolidWorks-exported per-wheel inertials had tiny (1e-8) off-diagonal
+    asymmetries that made the robot curve when commanded straight in Gazebo.
+  -->
   <link
     name="left_wheel_link">
     <inertial>
-      <origin
-        xyz="6.28502999154333E-07 -0.0039870676124848 -0.000569790977384271"
-        rpy="0 0 0" />
-      <mass
-        value="1.06112497715273" />
-      <inertia
-        ixx="0.00339900487986557"
-        ixy="-1.58838850523255E-08"
-        ixz="-5.99560271951721E-08"
-        iyy="0.00642634969436629"
-        iyz="-1.66764633557271E-07"
-        izz="0.0033973895137008" />
+      <origin xyz="0 0 0" rpy="0 0 0" />
+      <mass value="1.06112497715273" />
+      <inertia
+        ixx="0.003398197" ixy="0" ixz="0"
+        iyy="0.006426349" iyz="0"
+        izz="0.003397389" />
     </inertial>
     <visual>
@@ -499,5 +523,5 @@
       <origin xyz="0 0 0" rpy="1.5707963 0 0"/>
       <geometry>
-        <cylinder radius="0.11" length="0.046"/>
+        <cylinder radius="0.10" length="0.046"/>
       </geometry>
     </collision>
@@ -520,16 +544,10 @@
     name="right_wheel_link">
     <inertial>
-      <origin
-        xyz="-6.2850299915387E-07 0.0039870676124848 -0.000569790977384271"
-        rpy="0 0 0" />
-      <mass
-        value="1.06112497715273" />
-      <inertia
-        ixx="0.00339900487986557"
-        ixy="-1.58838850523222E-08"
-        ixz="5.99560271951723E-08"
-        iyy="0.00642634969436629"
-        iyz="1.66764633557271E-07"
-        izz="0.0033973895137008" />
+      <origin xyz="0 0 0" rpy="0 0 0" />
+      <mass value="1.06112497715273" />
+      <inertia
+        ixx="0.003398197" ixy="0" ixz="0"
+        iyy="0.006426349" iyz="0"
+        izz="0.003397389" />
     </inertial>
     <visual>
@@ -550,5 +568,5 @@
       <origin xyz="0 0 0" rpy="1.5707963 0 0"/>
       <geometry>
-        <cylinder radius="0.11" length="0.046"/>
+        <cylinder radius="0.10" length="0.046"/>
       </geometry>
     </collision>
@@ -621,4 +639,24 @@
       xyz="0 0 0" />
   </joint>
+  <!--
+    Camera links.
+    camera_link is the physical camera frame (X forward, Y left, Z up).
+    camera_rgb_optical_frame is its image-coordinate counterpart (X right,
+    Y down, Z forward) — the convention apriltag_ros::solvePnP requires when
+    computing the AprilTag pose. The rotation rpy="-1.5708 0 -1.5708" applied
+    to the optical joint is the standard −π/2, 0, −π/2 mapping.
+  -->
+  <link name="camera_link"/>
+  <joint name="camera_joint" type="fixed">
+    <origin xyz="0.35 0 0.22" rpy="0 0 0"/>
+    <parent link="base_link"/>
+    <child link="camera_link"/>
+  </joint>
+  <link name="camera_rgb_optical_frame"/>
+  <joint name="camera_optical_joint" type="fixed">
+    <origin xyz="0 0 0" rpy="-1.5707963 0 -1.5707963"/>
+    <parent link="camera_link"/>
+    <child link="camera_rgb_optical_frame"/>
+  </joint>
   <xacro:include filename="gazebo_control.xacro" />
 </robot>
