Commit message: feat: add Gemini RGB-D camera simulation
Signed-off-by: vineeth <manthenavineeth333@gmail.com>

File: ros2/src/openamrobot_description/urdf/gazebo_control.xacro (robot description, xacro)
@@ -133,12 +133,47 @@
   <xacro:caster_gazebo prefix="br" />
   <!-- ── Link-level: camera_link — forward-facing RGB camera ──────── -->
-  <gazebo reference="camera_link">
-    <material>Gazebo/Black</material>
-    <sensor name="camera_sensor" type="camera">
-      <pose relative_to="camera_link">0 0 0 0 0 0</pose>
-      <topic>/rgb_image</topic>
-      <gz_frame_id>camera_optical_frame</gz_frame_id>
+  <xacro:if value="$(arg legacy_camera)">
+    <gazebo reference="camera_link">
+      <material>Gazebo/Black</material>
+      <sensor name="camera_sensor" type="camera">
+        <pose relative_to="camera_link">0 0 0 0 0 0</pose>
+        <topic>/rgb_image</topic>
+        <gz_frame_id>camera_optical_frame</gz_frame_id>
+        <update_rate>12</update_rate>
+        <camera>
+          <horizontal_fov>1.047</horizontal_fov>
+          <image>
+            <width>640</width>
+            <height>480</height>
+            <format>R8G8B8</format>
+          </image>
+          <clip>
+            <near>0.05</near>
+            <far>15.0</far>
+          </clip>
+          <noise>
+            <type>gaussian</type>
+            <mean>0.0</mean>
+            <stddev>0.005</stddev>
+          </noise>
+        </camera>
+        <always_on>true</always_on>
+        <visualize>false</visualize>
+      </sensor>
+    </gazebo>
+  </xacro:if>
+  <!-- Gemini RGB-D simulation sensor. This is an idealized Gazebo sensor;
+       mount pose, optical calibration, and RGB/depth baseline are TBD and
+       must not be interpreted as Gemini/A6 physical measurements. Gazebo's
+       native RGBD sensor publishes one shared camera_info and uses the same
+       optical_frame_id for its RGB and depth image headers. -->
+  <gazebo reference="base_camera_link">
+    <sensor name="gemini_rgbd_sensor" type="rgbd_camera">
+      <pose relative_to="base_camera_link">0 0 0 0 0 0</pose>
+      <topic>/base_camera/rgbd</topic>
+      <gz_frame_id>base_camera_color_optical_frame</gz_frame_id>
       <update_rate>12</update_rate>
       <camera>
+        <!-- Provisional simulation settings, using the existing sim camera profile. -->
         <horizontal_fov>1.047</horizontal_fov>
         <image>
@@ -151,9 +186,5 @@
           <far>15.0</far>
         </clip>
-        <noise>
-          <type>gaussian</type>
-          <mean>0.0</mean>
-          <stddev>0.005</stddev>
-        </noise>
+        <optical_frame_id>base_camera_color_optical_frame</optical_frame_id>
       </camera>
       <always_on>true</always_on>

Commit message: feat: add Gemini RGB-D camera simulation

File: ros2/src/openamrobot_description/urdf/gazebo_control.xacro (robot description, xacro)
@@ -154,4 +154,33 @@
     </sensor>
   </gazebo>
+  <!-- Gemini RGB-D simulation sensor. This is an idealized Gazebo sensor;
+       mount pose, optical calibration, and RGB/depth baseline are TBD and
+       must not be interpreted as Gemini/A6 physical measurements. Gazebo's
+       native RGBD sensor publishes one shared camera_info and uses the same
+       optical_frame_id for its RGB and depth image headers. -->
+  <gazebo reference="base_camera_link">
+    <sensor name="gemini_rgbd_sensor" type="rgbd_camera">
+      <pose relative_to="base_camera_link">0 0 0 0 0 0</pose>
+      <topic>/base_camera/rgbd</topic>
+      <gz_frame_id>base_camera_color_optical_frame</gz_frame_id>
+      <update_rate>12</update_rate>
+      <camera>
+        <!-- Provisional simulation settings, using the existing sim camera profile. -->
+        <horizontal_fov>1.047</horizontal_fov>
+        <image>
+          <width>640</width>
+          <height>480</height>
+          <format>R8G8B8</format>
+        </image>
+        <clip>
+          <near>0.05</near>
+          <far>15.0</far>
+        </clip>
+        <optical_frame_id>base_camera_color_optical_frame</optical_frame_id>
+      </camera>
+      <always_on>true</always_on>
+      <visualize>false</visualize>
+    </sensor>
+  </gazebo>
   <!-- ── Link-level: lidar_link — sensor ONLY here ─────────────────── -->
   <gazebo reference="lidar_link">

File: ros2/src/openamrobot_description/urdf/robo_urdf.urdf.xacro (robot description, xacro)
@@ -655,4 +655,31 @@
     <child link="camera_optical_frame"/>
   </joint>
+  <!-- Gemini RGB-D assembly. Z = 0.143 m is derived from the current baseline
+       lens floor height (~0.243 m) and base_link floor reference (~0.100 m).
+       X remains a provisional simulation placeholder pending confirmation of
+       current bracket/hardware geometry; Y = 0 m places it on the centreline.
+       The -0.1745 rad pitch is the confirmed baseline 10-degree up-tilt.
+       This provisional origin is not claimed as final physical calibration. -->
+  <link name="base_camera_link"/>
+  <joint name="base_camera_joint" type="fixed">
+    <origin xyz="0 0 0.143" rpy="0 -0.1745 0"/>
+    <parent link="base_link"/>
+    <child link="base_camera_link"/>
+  </joint>
+  <!-- Optical axes: +Z forward, +X right, +Y down. The two optical origins
+       are temporarily co-located for simulation; the real RGB/depth baseline
+       and extrinsics remain TBD pending the Gemini camera geometry. -->
+  <link name="base_camera_color_optical_frame"/>
+  <joint name="base_camera_color_optical_joint" type="fixed">
+    <origin xyz="0 0 0" rpy="-1.5707963 0 -1.5707963"/>
+    <parent link="base_camera_link"/>
+    <child link="base_camera_color_optical_frame"/>
+  </joint>
+  <link name="base_camera_depth_optical_frame"/>
+  <joint name="base_camera_depth_optical_joint" type="fixed">
+    <origin xyz="0 0 0" rpy="-1.5707963 0 -1.5707963"/>
+    <parent link="base_camera_link"/>
+    <child link="base_camera_depth_optical_frame"/>
+  </joint>
   <xacro:include filename="gazebo_control.xacro" />
 </robot>

Commit message: feat: add Gemini RGB-D camera simulation
Signed-off-by: vineeth <manthenavineeth333@gmail.com>

File: ros2/src/openamrobot_description/urdf/gazebo_control.xacro (robot description, xacro)
@@ -133,12 +133,47 @@
   <xacro:caster_gazebo prefix="br" />
   <!-- ── Link-level: camera_link — forward-facing RGB camera ──────── -->
-  <gazebo reference="camera_link">
-    <material>Gazebo/Black</material>
-    <sensor name="camera_sensor" type="camera">
-      <pose relative_to="camera_link">0 0 0 0 0 0</pose>
-      <topic>/rgb_image</topic>
-      <gz_frame_id>camera_optical_frame</gz_frame_id>
+  <xacro:if value="$(arg legacy_camera)">
+    <gazebo reference="camera_link">
+      <material>Gazebo/Black</material>
+      <sensor name="camera_sensor" type="camera">
+        <pose relative_to="camera_link">0 0 0 0 0 0</pose>
+        <topic>/rgb_image</topic>
+        <gz_frame_id>camera_optical_frame</gz_frame_id>
+        <update_rate>12</update_rate>
+        <camera>
+          <horizontal_fov>1.047</horizontal_fov>
+          <image>
+            <width>640</width>
+            <height>480</height>
+            <format>R8G8B8</format>
+          </image>
+          <clip>
+            <near>0.05</near>
+            <far>15.0</far>
+          </clip>
+          <noise>
+            <type>gaussian</type>
+            <mean>0.0</mean>
+            <stddev>0.005</stddev>
+          </noise>
+        </camera>
+        <always_on>true</always_on>
+        <visualize>false</visualize>
+      </sensor>
+    </gazebo>
+  </xacro:if>
+  <!-- Gemini RGB-D simulation sensor. This is an idealized Gazebo sensor;
+       mount pose, optical calibration, and RGB/depth baseline are TBD and
+       must not be interpreted as Gemini/A6 physical measurements. Gazebo's
+       native RGBD sensor publishes one shared camera_info and uses the same
+       optical_frame_id for its RGB and depth image headers. -->
+  <gazebo reference="base_camera_link">
+    <sensor name="gemini_rgbd_sensor" type="rgbd_camera">
+      <pose relative_to="base_camera_link">0 0 0 0 0 0</pose>
+      <topic>/base_camera/rgbd</topic>
+      <gz_frame_id>base_camera_color_optical_frame</gz_frame_id>
       <update_rate>12</update_rate>
       <camera>
+        <!-- Provisional simulation settings, using the existing sim camera profile. -->
         <horizontal_fov>1.047</horizontal_fov>
         <image>
@@ -151,9 +186,5 @@
           <far>15.0</far>
         </clip>
-        <noise>
-          <type>gaussian</type>
-          <mean>0.0</mean>
-          <stddev>0.005</stddev>
-        </noise>
+        <optical_frame_id>base_camera_color_optical_frame</optical_frame_id>
       </camera>
       <always_on>true</always_on>

File: ros2/src/openamrobot_description/urdf/robo_urdf.urdf.xacro (robot description, xacro)
@@ -708,4 +708,7 @@
        An unknown base_tilt value fails the xacro expansion. -->
   <xacro:arg name="base_tilt" default="bt10"/>
+  <!-- Legacy Gate A IMX708 simulation sensor selection; camera frames remain
+       available for existing docking and perception consumers. -->
+  <xacro:arg name="legacy_camera" default="false"/>
   <xacro:property name="base_camera_pitch"
     value="${dict(bt05=-0.0873, bt10=-0.1745, bt15=-0.2618)['$(arg base_tilt)']}"/>

Commit message: description: IMU at 165.043 mm above the base plate, 222.05 mm scan plane, Gazebo IMU (#49)
- imu_link (0.0544, 0, 0.1210), yaw -90 deg: ICM-42688-P package centre,
  165.043 mm above the base-plate top (219.04 mm above the floor).
- Scan plane 222.05 mm in the datum table, URDF/SDF comments and TF docs;
  lidar_link stays (0.330, 0, 0.124), yaw pi.
- Gazebo IMU sensor on imu_link and the gz-sim-imu-system plugin, copied from
  #69.

Signed-off-by: Cuma Ali Karaaslan <115656544+fridayali@users.noreply.github.com>

File: ros2/src/openamrobot_description/urdf/gazebo_control.xacro (robot description, xacro)
@@ -161,4 +161,25 @@
     </sensor>
   </gazebo>
+  <!-- ── Link-level: imu_link — simulated IMU (from #69) ─────────────── -->
+  <!-- Publishes gz topic "imu", which config/gz_bridge.yaml bridges to /imu.
+       The sensor sits on imu_link with no pose offset; the frame (sensor axes,
+       yaw -90 deg) is declared in sensors.xacro. The rate matches the 0.02 s
+       nominal period in openamrobot_nav2 navigation_status_profile.yaml. No noise
+       model: simulation only, not the ICM-42688-P's characteristics. -->
+  <gazebo reference="imu_link">
+    <sensor name="imu_sensor" type="imu">
+      <pose relative_to="imu_link">0 0 0 0 0 0</pose>
+      <topic>imu</topic>
+      <gz_frame_id>imu_link</gz_frame_id>
+      <update_rate>50</update_rate>
+      <always_on>true</always_on>
+      <visualize>false</visualize>
+    </sensor>
+  </gazebo>
+  <!-- The IMU system updates every imu sensor; neither walled_world.sdf nor
+       a world that composes this model loads it, so the model does. -->
+  <gazebo>
+    <plugin filename="gz-sim-imu-system" name="gz::sim::systems::Imu"/>
+  </gazebo>
   <!-- ── Link-level: lidar_link — sensor ONLY here ─────────────────── -->
   <gazebo reference="lidar_link">

File: ros2/src/openamrobot_description/urdf/robo_urdf.urdf.xacro (robot description, xacro)
@@ -640,5 +640,7 @@
     name="lidar_joint"
     type="fixed">
-    <!-- lidar_link origin at the scan-plane centre, 222.0 mm above the floor
+    <!-- lidar_link origin at the scan-plane centre, 222.05 mm above the floor
+         (MMP.07 bracket + 17.5 mm spacer, no standoffs; Alex decision 2026-10-16;
+         z 0.124 rounds it to 222.0 mm)
          (0.098 + 0.124), mounted rotated 180 deg (Alex decision 2026-10-12,
          STEP MMP.00.00.00.000). Superseded by Alex decision 2026-10-12:

File: ros2/src/openamrobot_description/urdf/sensors.xacro (robot description, xacro)
@@ -52,15 +52,15 @@
   <!-- IMU, ICM-42688-P on the MIKROE-4237 Click board, electronics bracket
        MMP.04.00.00.002. Origin at the centre of the ICM-42688-P package: on the
-       centreline, 54.4 mm in front of the drive axle, 222.6 mm above the floor
-       (168.6 mm above the base-plate top), CAD Rev B 2026-10-16.
+       centreline, 54.4 mm in front of the drive axle, 165.043 mm above the
+       base-plate top (54.0 mm), i.e. 219.04 mm above the floor (CAD 2026-10-16).
        Orientation: board flat, component side up, pin 1 at the front-left corner;
        sensor X -> base -y, Y -> +x, Z -> +z, so yaw -90 deg (datasheet axis check
        by Evans, CAD check 2026-10-16). imu_link is the sensor frame; the firmware
-       must not remap the axes as well.
-       Was (0.0544, 0, 0.133) rpy 0 (16 Oct: 177 mm was measured against a
+       publishes in it and must not remap the axes as well.
+       Was (0.0544, 0, 0.133) rpy 0 (16 Oct; 177 mm was measured against a
        displaced base plate) and (0.195, 0, -0.044) (Alex decision 2026-10-12). -->
   <link name="imu_link"/>
   <joint name="imu_joint" type="fixed">
-    <origin xyz="0.0544 0 0.1246" rpy="0 0 ${-pi/2}"/>
+    <origin xyz="0.0544 0 0.1210" rpy="0 0 ${-pi/2}"/>
     <parent link="base_link"/>
     <child link="imu_link"/>
