Commit message: fix(sim): restore simulation after restructuring regressions
- gz_simulator.launch.py: remove standalone joint_state_publisher node;
  it conflicted with gz-sim-joint-state-publisher-system (both
  publishing /joint_states), causing wheel TF flicker in RViz.
- robo_urdf.urdf.xacro: restore wheel collision cylinder radius to
  0.11 m. The DiffDrive plugin kinematic wheel_radius (0.10 m) is
  independent from the collision geometry; with the cylinder at 0.10
  the wheels only touched the ground (zero penetration -> zero normal
  force -> zero friction) and the robot could not move.
- apriltag_sim.launch.yml: fix tags_36h11_sim.yaml path after
  config/ flattening. The launch still referenced the old
  simulation/config/ location and the detector silently started
  with no tag declared.

File: ros2/src/openamrobot_description/urdf/robo_urdf.urdf.xacro (robot description, xacro)
@@ -523,5 +523,9 @@
       <origin xyz="0 0 0" rpy="1.5707963 0 0"/>
       <geometry>
-        <cylinder radius="0.10" length="0.046"/>
+        <!-- 0.11 cylinder vs DiffDrive wheel_radius=0.10 gives ~1 cm of
+             penetration into the ground plane, which ODE's contact solver
+             uses to apply traction. Without that overlap the wheels merely
+             touch the floor and the robot does not move. -->
+        <cylinder radius="0.11" length="0.046"/>
       </geometry>
     </collision>
@@ -568,5 +572,9 @@
       <origin xyz="0 0 0" rpy="1.5707963 0 0"/>
       <geometry>
-        <cylinder radius="0.10" length="0.046"/>
+        <!-- 0.11 cylinder vs DiffDrive wheel_radius=0.10 gives ~1 cm of
+             penetration into the ground plane, which ODE's contact solver
+             uses to apply traction. Without that overlap the wheels merely
+             touch the floor and the robot does not move. -->
+        <cylinder radius="0.11" length="0.046"/>
       </geometry>
     </collision>
