Commit message: description: 2.0 sensor frames from CAD v0.2 and simplified collision (#49)
- Sensor links and joints in urdf/sensors.xacro, included by the main xacro.
  Poses from the OpenAMRobot platform v0.2 CAD; each frame with its CAD source
  and status in config/sensor_frames.yaml.
- Four TF-Luna (tof_front_left/right, tof_rear_left/right, 10 deg down) and two
  MB7060 (us_front, us_rear) replace us_front_left/right, us_rear_left/right,
  tof_front and tof_rear.
- base_camera_link (Gemini 336L) at (0.386, 0, 0.0447) on the 10 deg mount;
  base_tilt gains bt00, default stays bt10.
- Collision: chassis, castors and LiDAR are boxes/cylinders instead of STL
  meshes; the A1 LiDAR mesh is replaced with an RPLIDAR S3 cylinder.
- Gazebo range sensors on /tof/* and /ultrasonic/*, bridged as LaserScan.
- robot.sdf, docs and CHANGELOG updated. imu_link stays a placeholder until the
  IMU plate is designed.

check_urdf passes for base_tilt bt00/bt05/bt10/bt15.

Signed-off-by: Cuma Ali Karaaslan <115656544+fridayali@users.noreply.github.com>

File: ros2/src/openamrobot_description/urdf/robo_urdf.urdf.xacro (robot description, xacro)
@@ -57,12 +57,10 @@
     </visual>
     <collision>
-      <!-- legacy mesh kept at its floor height: z -0.034533 (Alex decision 2026-10-12);
-           was xyz="0 0 0", superseded by Alex decision 2026-10-12 -->
-      <origin
-        xyz="0 0 -0.034533"
-        rpy="0 0 0" />
-      <geometry>
-        <mesh
-          filename="package://openamrobot_description/meshes/visual/base_link.STL" />
+      <!-- Chassis box, CAD Rev B STEP MMP.00.00.00.000: x +-0.390 (panel faces),
+           y +-0.290 (base plate), 0.050 to 0.295 m above the floor (panel bottom to
+           cover top). Was the base_link.STL visual mesh, superseded (#49). -->
+      <origin xyz="0 0 0.0745" rpy="0 0 0"/>
+      <geometry>
+        <box size="0.780 0.580 0.245"/>
       </geometry>
     </collision>
@@ -99,10 +97,9 @@
     </visual>
     <collision>
-      <origin
-        xyz="0 0 0"
-        rpy="0 0 0" />
-      <geometry>
-        <mesh
-          filename="package://openamrobot_description/meshes/visual/fl_caster_link.STL" />
+      <!-- Castor housing GH-LPA035 0.060 x 0.060 m, 0.0125 to 0.052 m above the
+           floor (CAD Rev B). Was the caster STL mesh, superseded (#49). -->
+      <origin xyz="0 0 -0.022" rpy="0 0 0"/>
+      <geometry>
+        <box size="0.060 0.060 0.040"/>
       </geometry>
     </collision>
@@ -206,10 +203,9 @@
     </visual>
     <collision>
-      <origin
-        xyz="0 0 0"
-        rpy="0 0 0" />
-      <geometry>
-        <mesh
-          filename="package://openamrobot_description/meshes/visual/fr_caster_link.STL" />
+      <!-- Castor housing GH-LPA035 0.060 x 0.060 m, 0.0125 to 0.052 m above the
+           floor (CAD Rev B). Was the caster STL mesh, superseded (#49). -->
+      <origin xyz="0 0 -0.022" rpy="0 0 0"/>
+      <geometry>
+        <box size="0.060 0.060 0.040"/>
       </geometry>
     </collision>
@@ -313,10 +309,9 @@
     </visual>
     <collision>
-      <origin
-        xyz="0 0 0"
-        rpy="0 0 0" />
-      <geometry>
-        <mesh
-          filename="package://openamrobot_description/meshes/visual/br_caster_link.STL" />
+      <!-- Castor housing GH-LPA035 0.060 x 0.060 m, 0.0125 to 0.052 m above the
+           floor (CAD Rev B). Was the caster STL mesh, superseded (#49). -->
+      <origin xyz="0 0 -0.022" rpy="0 0 0"/>
+      <geometry>
+        <box size="0.060 0.060 0.040"/>
       </geometry>
     </collision>
@@ -420,10 +415,9 @@
     </visual>
     <collision>
-      <origin
-        xyz="0 0 0"
-        rpy="0 0 0" />
-      <geometry>
-        <mesh
-          filename="package://openamrobot_description/meshes/visual/bl_caster_link.STL" />
+      <!-- Castor housing GH-LPA035 0.060 x 0.060 m, 0.0125 to 0.052 m above the
+           floor (CAD Rev B). Was the caster STL mesh, superseded (#49). -->
+      <origin xyz="0 0 -0.022" rpy="0 0 0"/>
+      <geometry>
+        <box size="0.060 0.060 0.040"/>
       </geometry>
     </collision>
@@ -624,25 +618,20 @@
         izz="0.000100924865484583" />
     </inertial>
-    <visual>
-      <origin
-        xyz="0 0 0"
-        rpy="0 0 0" />
-      <geometry>
-        <mesh
-          filename="package://openamrobot_description/meshes/visual/lidar_link.STL" />
-      </geometry>
-      <material
-        name="">
-        <color
-          rgba="0.792156862745098 0.819607843137255 0.933333333333333 1" />
-      </material>
-    </visual>
-    <collision>
-      <origin
-        xyz="0 0 0"
-        rpy="0 0 0" />
-      <geometry>
-        <mesh
-          filename="package://openamrobot_description/meshes/visual/lidar_link.STL" />
+    <!-- RPLIDAR S3 body: cylinder 0.0556 m diameter, 0.0413 m high, 0.0277 m below
+         to 0.0136 m above the scan plane (CAD Rev B). Was the A1 lidar_link.STL
+         mesh, superseded (#49). The inertial above is still the A1 one. -->
+    <visual>
+      <origin xyz="0 0 -0.00765" rpy="0 0 0"/>
+      <geometry>
+        <cylinder radius="0.0278" length="0.0413"/>
+      </geometry>
+      <material name="lidar_black">
+        <color rgba="0.1 0.1 0.1 1"/>
+      </material>
+    </visual>
+    <collision>
+      <origin xyz="0 0 -0.00765" rpy="0 0 0"/>
+      <geometry>
+        <cylinder radius="0.0278" length="0.0413"/>
       </geometry>
     </collision>
@@ -655,5 +644,6 @@
          STEP MMP.00.00.00.000). Superseded by Alex decision 2026-10-12:
          xyz="0.35135 -0.0010251 0.1683" rpy="0 0 0". The lidar visual/collision
-         mesh is the legacy A1 mesh and is not re-placed by this change. -->
+         shape is the RPLIDAR S3 cylinder (#49). CAD Rev B places the S3 centre
+         at x 0.321; lidar_link is kept at 0.330 until that is decided. -->
     <origin
       xyz="0.330 0 0.124"
@@ -702,62 +692,6 @@
     <child link="camera_optical_frame"/>
   </joint>
-  <!-- ── OpenAMRobot 2.0 sensor frames (Alex decision 2026-10-12) ────── -->
-  <!-- Base camera, Orbbec Gemini 336L. Tilt is a configuration ID:
-       base_tilt:=bt05 / bt10 / bt15 -> pitch -0.0873 / -0.1745 / -0.2618 rad
-       (5 / 10 / 15 deg up), default bt10 (Alex decision 2026-10-12).
-       An unknown base_tilt value fails the xacro expansion. -->
-  <xacro:arg name="base_tilt" default="bt10"/>
-  <xacro:property name="base_camera_pitch"
-    value="${dict(bt05=-0.0873, bt10=-0.1745, bt15=-0.2618)['$(arg base_tilt)']}"/>
-  <link name="base_camera_link"/>
-  <!-- xyz (0.376, 0, 0.0445) (Alex decision 2026-10-12, STEP MMP.00.00.00.000) -->
-  <joint name="base_camera_joint" type="fixed">
-    <origin xyz="0.376 0 0.0445" rpy="0 ${base_camera_pitch} 0"/>
-    <parent link="base_link"/>
-    <child link="base_camera_link"/>
-  </joint>
-  <!-- Optical frames: ROS optical convention, z forward, x right, y down
-       (Alex decision 2026-10-12) -->
-  <link name="base_camera_color_optical_frame"/>
-  <joint name="base_camera_color_optical_joint" type="fixed">
-    <origin xyz="0 0 0" rpy="${-pi/2} 0 ${-pi/2}"/>
-    <parent link="base_camera_link"/>
-    <child link="base_camera_color_optical_frame"/>
-  </joint>
-  <link name="base_camera_depth_optical_frame"/>
-  <joint name="base_camera_depth_optical_joint" type="fixed">
-    <origin xyz="0 0 0" rpy="${-pi/2} 0 ${-pi/2}"/>
-    <parent link="base_camera_link"/>
-    <child link="base_camera_depth_optical_frame"/>
-  </joint>
-  <!-- IMU, ICM-42688-P: xyz (0.195, 0, -0.044), rpy 0 (Alex decision 2026-10-12,
-       STEP MMP.00.00.00.000). base plate top; board stack height added from the
-       mount drawing. -->
-  <link name="imu_link"/>
-  <joint name="imu_joint" type="fixed">
-    <origin xyz="0.195 0 -0.044" rpy="0 0 0"/>
-    <parent link="base_link"/>
-    <child link="imu_link"/>
-  </joint>
-  <!-- Near-field sensors at the panel hole centres, fixed to base_link
-       (Alex decision 2026-10-12, STEP MMP.00.00.00.000). -->
-  <xacro:macro name="near_field_frame" params="name x y z pitch:=0 yaw:=0">
-    <link name="${name}"/>
-    <joint name="${name}_joint" type="fixed">
-      <origin xyz="${x} ${y} ${z}" rpy="0 ${pitch} ${yaw}"/>
-      <parent link="base_link"/>
-      <child link="${name}"/>
-    </joint>
-  </xacro:macro>
-  <!-- Ultrasonic, MB7060 (Alex decision 2026-10-12, STEP MMP.00.00.00.000) -->
-  <xacro:near_field_frame name="us_front_left" x="0.390" y="0.130" z="-0.0066"/>
-  <xacro:near_field_frame name="us_front_right" x="0.390" y="-0.130" z="-0.0066"/>
-  <xacro:near_field_frame name="us_rear_left" x="-0.390" y="0.130" z="-0.0066" yaw="${pi}"/>
-  <xacro:near_field_frame name="us_rear_right" x="-0.390" y="-0.130" z="-0.0066" yaw="${pi}"/>
-  <!-- ToF, TF-Luna (Alex decision 2026-10-12, STEP MMP.00.00.00.000).
-       20 degree down screening value until the bench test. -->
-  <xacro:near_field_frame name="tof_front" x="0.390" y="0" z="-0.0066" pitch="0.3491"/>
-  <!-- 20 degree down screening value until the bench test. -->
-  <xacro:near_field_frame name="tof_rear" x="-0.390" y="0" z="-0.0066" pitch="0.3491" yaw="${pi}"/>
+  <!-- OpenAMRobot 2.0 sensor frames: Gemini 336L, IMU, TF-Luna, MB7060 (#49) -->
+  <xacro:include filename="sensors.xacro" />
   <xacro:include filename="gazebo_control.xacro" />
 </robot>

Commit message: fix: update Gemini base camera mounting pose
Signed-off-by: vineeth <manthenavineeth333@gmail.com>

File: ros2/src/openamrobot_description/urdf/robo_urdf.urdf.xacro (robot description, xacro)
@@ -714,7 +714,7 @@
     value="${dict(bt05=-0.0873, bt10=-0.1745, bt15=-0.2618)['$(arg base_tilt)']}"/>
   <link name="base_camera_link"/>
-  <!-- xyz (0.376, 0, 0.0445) (Alex decision 2026-10-12, STEP MMP.00.00.00.000) -->
+  <!-- xyz (0.387, 0, 0.046) (Gemini 336L base-camera mounting position) -->
   <joint name="base_camera_joint" type="fixed">
-    <origin xyz="0.376 0 0.0445" rpy="0 ${base_camera_pitch} 0"/>
+    <origin xyz="0.387 0 0.046" rpy="0 ${base_camera_pitch} 0"/>
     <parent link="base_link"/>
     <child link="base_camera_link"/>

Commit message: description: 2.0 sensor frames, simplified collision and Gazebo sensors (#49) (#70)
* description: 2.0 sensor frames from CAD v0.2 and simplified collision (#49)

- Sensor links and joints in urdf/sensors.xacro, included by the main xacro.
  Poses from the OpenAMRobot platform v0.2 CAD; each frame with its CAD source
  and status in config/sensor_frames.yaml.
- Four TF-Luna (tof_front_left/right, tof_rear_left/right, 10 deg down) and two
  MB7060 (us_front, us_rear) replace us_front_left/right, us_rear_left/right,
  tof_front and tof_rear.
- base_camera_link (Gemini 336L) at (0.386, 0, 0.0447) on the 10 deg mount;
  base_tilt gains bt00, default stays bt10.
- Collision: chassis, castors and LiDAR are boxes/cylinders instead of STL
  meshes; the A1 LiDAR mesh is replaced with an RPLIDAR S3 cylinder.
- Gazebo range sensors on /tof/* and /ultrasonic/*, bridged as LaserScan.
- robot.sdf, docs and CHANGELOG updated. imu_link stays a placeholder until the
  IMU plate is designed.

check_urdf passes for base_tilt bt00/bt05/bt10/bt15.

Signed-off-by: Cuma Ali Karaaslan <115656544+fridayali@users.noreply.github.com>

* description: decided sensor layout (P-03 rev19.0 item 19) and Rev B CAD poses (#49)

- 4 x MB7060 (us_front_left/right, us_rear_left/right) at y +-0.130 and
  2 x TF-Luna (tof_front, tof_rear, 20 deg down screening value); existing
  link and joint names kept.
- base_camera_link (0.387, 0, 0.046) and imu_link (0.0544, 0, 0.133) from the
  CAD Rev B full assembly (2026-10-15); base_tilt bt05/bt10/bt15, bt00 removed.
- sensor_frames.yaml, robot.sdf, gz_bridge topics, TF docs and CHANGELOG
  updated; LiDAR stack note: MMP.07 bracket + 17.5 mm spacer, beam 222.05 mm.

Signed-off-by: Cuma Ali Karaaslan <115656544+fridayali@users.noreply.github.com>

* description: imu_link at the ICM-42688-P package centre, yaw -90 deg (#49)

- imu_link (0.0544, 0, 0.1246): ICM-42688-P package centre on the electronics
  bracket, 222.6 mm above the floor, 168.6 mm above the base-plate top (CAD
  2026-10-16). The 16 Oct 0.133 came from 177 mm measured against a displaced
  base plate in the CAD.
- rpy (0, 0, -pi/2): board flat, component side up, pin 1 front-left; sensor
  X -> base -y, Y -> +x, Z -> +z (datasheet axis check by Evans, CAD check).
  imu_link is the sensor frame; the firmware must not remap the axes too.
- sensor_frames.yaml, robot.sdf, TF docs and CHANGELOG updated.

check_urdf passes for base_tilt bt05/bt10/bt15.

Signed-off-by: Cuma Ali Karaaslan <115656544+fridayali@users.noreply.github.com>

* description: IMU at 165.043 mm above the base plate, 222.05 mm scan plane, Gazebo IMU (#49)

- imu_link (0.0544, 0, 0.1210), yaw -90 deg: ICM-42688-P package centre,
  165.043 mm above the base-plate top (219.04 mm above the floor).
- Scan plane 222.05 mm in the datum table, URDF/SDF comments and TF docs;
  lidar_link stays (0.330, 0, 0.124), yaw pi.
- Gazebo IMU sensor on imu_link and the gz-sim-imu-system plugin, copied from
  #69.

Signed-off-by: Cuma Ali Karaaslan <115656544+fridayali@users.noreply.github.com>

---------

Signed-off-by: Cuma Ali Karaaslan <115656544+fridayali@users.noreply.github.com>

File: ros2/src/openamrobot_description/urdf/robo_urdf.urdf.xacro (robot description, xacro)
@@ -57,12 +57,10 @@
     </visual>
     <collision>
-      <!-- legacy mesh kept at its floor height: z -0.034533 (Alex decision 2026-10-12);
-           was xyz="0 0 0", superseded by Alex decision 2026-10-12 -->
-      <origin
-        xyz="0 0 -0.034533"
-        rpy="0 0 0" />
-      <geometry>
-        <mesh
-          filename="package://openamrobot_description/meshes/visual/base_link.STL" />
+      <!-- Chassis box, CAD Rev B STEP MMP.00.00.00.000: x +-0.390 (panel faces),
+           y +-0.290 (base plate), 0.050 to 0.295 m above the floor (panel bottom to
+           cover top). Was the base_link.STL visual mesh, superseded (#49). -->
+      <origin xyz="0 0 0.0745" rpy="0 0 0"/>
+      <geometry>
+        <box size="0.780 0.580 0.245"/>
       </geometry>
     </collision>
@@ -99,10 +97,9 @@
     </visual>
     <collision>
-      <origin
-        xyz="0 0 0"
-        rpy="0 0 0" />
-      <geometry>
-        <mesh
-          filename="package://openamrobot_description/meshes/visual/fl_caster_link.STL" />
+      <!-- Castor housing GH-LPA035 0.060 x 0.060 m, 0.0125 to 0.052 m above the
+           floor (CAD Rev B). Was the caster STL mesh, superseded (#49). -->
+      <origin xyz="0 0 -0.022" rpy="0 0 0"/>
+      <geometry>
+        <box size="0.060 0.060 0.040"/>
       </geometry>
     </collision>
@@ -206,10 +203,9 @@
     </visual>
     <collision>
-      <origin
-        xyz="0 0 0"
-        rpy="0 0 0" />
-      <geometry>
-        <mesh
-          filename="package://openamrobot_description/meshes/visual/fr_caster_link.STL" />
+      <!-- Castor housing GH-LPA035 0.060 x 0.060 m, 0.0125 to 0.052 m above the
+           floor (CAD Rev B). Was the caster STL mesh, superseded (#49). -->
+      <origin xyz="0 0 -0.022" rpy="0 0 0"/>
+      <geometry>
+        <box size="0.060 0.060 0.040"/>
       </geometry>
     </collision>
@@ -313,10 +309,9 @@
     </visual>
     <collision>
-      <origin
-        xyz="0 0 0"
-        rpy="0 0 0" />
-      <geometry>
-        <mesh
-          filename="package://openamrobot_description/meshes/visual/br_caster_link.STL" />
+      <!-- Castor housing GH-LPA035 0.060 x 0.060 m, 0.0125 to 0.052 m above the
+           floor (CAD Rev B). Was the caster STL mesh, superseded (#49). -->
+      <origin xyz="0 0 -0.022" rpy="0 0 0"/>
+      <geometry>
+        <box size="0.060 0.060 0.040"/>
       </geometry>
     </collision>
@@ -420,10 +415,9 @@
     </visual>
     <collision>
-      <origin
-        xyz="0 0 0"
-        rpy="0 0 0" />
-      <geometry>
-        <mesh
-          filename="package://openamrobot_description/meshes/visual/bl_caster_link.STL" />
+      <!-- Castor housing GH-LPA035 0.060 x 0.060 m, 0.0125 to 0.052 m above the
+           floor (CAD Rev B). Was the caster STL mesh, superseded (#49). -->
+      <origin xyz="0 0 -0.022" rpy="0 0 0"/>
+      <geometry>
+        <box size="0.060 0.060 0.040"/>
       </geometry>
     </collision>
@@ -624,25 +618,20 @@
         izz="0.000100924865484583" />
     </inertial>
-    <visual>
-      <origin
-        xyz="0 0 0"
-        rpy="0 0 0" />
-      <geometry>
-        <mesh
-          filename="package://openamrobot_description/meshes/visual/lidar_link.STL" />
-      </geometry>
-      <material
-        name="">
-        <color
-          rgba="0.792156862745098 0.819607843137255 0.933333333333333 1" />
-      </material>
-    </visual>
-    <collision>
-      <origin
-        xyz="0 0 0"
-        rpy="0 0 0" />
-      <geometry>
-        <mesh
-          filename="package://openamrobot_description/meshes/visual/lidar_link.STL" />
+    <!-- RPLIDAR S3 body: cylinder 0.0556 m diameter, 0.0413 m high, 0.0277 m below
+         to 0.0136 m above the scan plane (CAD Rev B). Was the A1 lidar_link.STL
+         mesh, superseded (#49). The inertial above is still the A1 one. -->
+    <visual>
+      <origin xyz="0 0 -0.00765" rpy="0 0 0"/>
+      <geometry>
+        <cylinder radius="0.0278" length="0.0413"/>
+      </geometry>
+      <material name="lidar_black">
+        <color rgba="0.1 0.1 0.1 1"/>
+      </material>
+    </visual>
+    <collision>
+      <origin xyz="0 0 -0.00765" rpy="0 0 0"/>
+      <geometry>
+        <cylinder radius="0.0278" length="0.0413"/>
       </geometry>
     </collision>
@@ -651,9 +640,12 @@
     name="lidar_joint"
     type="fixed">
-    <!-- lidar_link origin at the scan-plane centre, 222.0 mm above the floor
+    <!-- lidar_link origin at the scan-plane centre, 222.05 mm above the floor
+         (MMP.07 bracket + 17.5 mm spacer, no standoffs; Alex decision 2026-10-16;
+         z 0.124 rounds it to 222.0 mm)
          (0.098 + 0.124), mounted rotated 180 deg (Alex decision 2026-10-12,
          STEP MMP.00.00.00.000). Superseded by Alex decision 2026-10-12:
          xyz="0.35135 -0.0010251 0.1683" rpy="0 0 0". The lidar visual/collision
-         mesh is the legacy A1 mesh and is not re-placed by this change. -->
+         shape is the RPLIDAR S3 cylinder (#49). CAD Rev B places the S3 centre
+         at x 0.321; lidar_link is kept at 0.330 until that is decided. -->
     <origin
       xyz="0.330 0 0.124"
@@ -702,62 +694,6 @@
     <child link="camera_optical_frame"/>
   </joint>
-  <!-- ── OpenAMRobot 2.0 sensor frames (Alex decision 2026-10-12) ────── -->
-  <!-- Base camera, Orbbec Gemini 336L. Tilt is a configuration ID:
-       base_tilt:=bt05 / bt10 / bt15 -> pitch -0.0873 / -0.1745 / -0.2618 rad
-       (5 / 10 / 15 deg up), default bt10 (Alex decision 2026-10-12).
-       An unknown base_tilt value fails the xacro expansion. -->
-  <xacro:arg name="base_tilt" default="bt10"/>
-  <xacro:property name="base_camera_pitch"
-    value="${dict(bt05=-0.0873, bt10=-0.1745, bt15=-0.2618)['$(arg base_tilt)']}"/>
-  <link name="base_camera_link"/>
-  <!-- xyz (0.376, 0, 0.0445) (Alex decision 2026-10-12, STEP MMP.00.00.00.000) -->
-  <joint name="base_camera_joint" type="fixed">
-    <origin xyz="0.376 0 0.0445" rpy="0 ${base_camera_pitch} 0"/>
-    <parent link="base_link"/>
-    <child link="base_camera_link"/>
-  </joint>
-  <!-- Optical frames: ROS optical convention, z forward, x right, y down
-       (Alex decision 2026-10-12) -->
-  <link name="base_camera_color_optical_frame"/>
-  <joint name="base_camera_color_optical_joint" type="fixed">
-    <origin xyz="0 0 0" rpy="${-pi/2} 0 ${-pi/2}"/>
-    <parent link="base_camera_link"/>
-    <child link="base_camera_color_optical_frame"/>
-  </joint>
-  <link name="base_camera_depth_optical_frame"/>
-  <joint name="base_camera_depth_optical_joint" type="fixed">
-    <origin xyz="0 0 0" rpy="${-pi/2} 0 ${-pi/2}"/>
-    <parent link="base_camera_link"/>
-    <child link="base_camera_depth_optical_frame"/>
-  </joint>
-  <!-- IMU, ICM-42688-P: xyz (0.195, 0, -0.044), rpy 0 (Alex decision 2026-10-12,
-       STEP MMP.00.00.00.000). base plate top; board stack height added from the
-       mount drawing. -->
-  <link name="imu_link"/>
-  <joint name="imu_joint" type="fixed">
-    <origin xyz="0.195 0 -0.044" rpy="0 0 0"/>
-    <parent link="base_link"/>
-    <child link="imu_link"/>
-  </joint>
-  <!-- Near-field sensors at the panel hole centres, fixed to base_link
-       (Alex decision 2026-10-12, STEP MMP.00.00.00.000). -->
-  <xacro:macro name="near_field_frame" params="name x y z pitch:=0 yaw:=0">
-    <link name="${name}"/>
-    <joint name="${name}_joint" type="fixed">
-      <origin xyz="${x} ${y} ${z}" rpy="0 ${pitch} ${yaw}"/>
-      <parent link="base_link"/>
-      <child link="${name}"/>
-    </joint>
-  </xacro:macro>
-  <!-- Ultrasonic, MB7060 (Alex decision 2026-10-12, STEP MMP.00.00.00.000) -->
-  <xacro:near_field_frame name="us_front_left" x="0.390" y="0.130" z="-0.0066"/>
-  <xacro:near_field_frame name="us_front_right" x="0.390" y="-0.130" z="-0.0066"/>
-  <xacro:near_field_frame name="us_rear_left" x="-0.390" y="0.130" z="-0.0066" yaw="${pi}"/>
-  <xacro:near_field_frame name="us_rear_right" x="-0.390" y="-0.130" z="-0.0066" yaw="${pi}"/>
-  <!-- ToF, TF-Luna (Alex decision 2026-10-12, STEP MMP.00.00.00.000).
-       20 degree down screening value until the bench test. -->
-  <xacro:near_field_frame name="tof_front" x="0.390" y="0" z="-0.0066" pitch="0.3491"/>
-  <!-- 20 degree down screening value until the bench test. -->
-  <xacro:near_field_frame name="tof_rear" x="-0.390" y="0" z="-0.0066" pitch="0.3491" yaw="${pi}"/>
+  <!-- OpenAMRobot 2.0 sensor frames: Gemini 336L, IMU, TF-Luna, MB7060 (#49) -->
+  <xacro:include filename="sensors.xacro" />
   <xacro:include filename="gazebo_control.xacro" />
 </robot>
