Commit message: description: imu_link at the CAD Rev B position (Alex decision 2026-10-16)
imu_link moves from (0.195, 0, -0.044) to (0.0544, 0, 0.133): ICM-42688-P on
the electronics bracket MMP.04.00.00.002 (platform-hw #20), on the centreline,
54.4 mm ahead of the drive axle, 177 mm above the base-plate top. This also
closes the open IMU board-stack height. Docs frame trees updated to match.

Co-Authored-By: Claude Opus 5.5 <noreply@anthropic.com>
Claude-Session: https://claude.ai/code/session_015uY6hFMbCNTirChFEieXEs
Signed-off-by: Alex Reznichenko <info@botshare.ai>

File: ros2/src/openamrobot_description/urdf/robo_urdf.urdf.xacro (robot description, xacro)
@@ -731,10 +731,12 @@
     <child link="base_camera_depth_optical_frame"/>
   </joint>
-  <!-- IMU, ICM-42688-P: xyz (0.195, 0, -0.044), rpy 0 (Alex decision 2026-10-12,
-       STEP MMP.00.00.00.000). base plate top; board stack height added from the
-       mount drawing. -->
+  <!-- IMU, ICM-42688-P: xyz (0.0544, 0, 0.133), rpy 0 (Alex decision 2026-10-16,
+       CAD Rev B, platform-hw #20): on the electronics bracket MMP.04.00.00.002, on
+       the centreline, 54.4 mm ahead of the drive axle, 177 mm above the base-plate
+       top (z -0.044 + 0.177). Supersedes (0.195, 0, -0.044) of 2026-10-12, which
+       had no board-stack height. Axes aligned with base_link. -->
   <link name="imu_link"/>
   <joint name="imu_joint" type="fixed">
-    <origin xyz="0.195 0 -0.044" rpy="0 0 0"/>
+    <origin xyz="0.0544 0 0.133" rpy="0 0 0"/>
     <parent link="base_link"/>
     <child link="imu_link"/>

Commit message: description: chassis collision box clears the caster wheels
The #70 chassis box (bottom 0.050 m above the floor) overlapped the four
caster-wheel collision spheres (top 0.0524 m) by 2.4 mm, a permanent
self-collision that fails the combined model's collision-matrix check (M03).
The box bottom moves to 0.055 m (top unchanged at 0.295 m): 2.6 mm clearance.
Found by the Jazzy check of main d619012 (issue #49).

Co-Authored-By: Claude Opus 5.5 <noreply@anthropic.com>
Claude-Session: https://claude.ai/code/session_015uY6hFMbCNTirChFEieXEs
Signed-off-by: Alex Reznichenko <info@botshare.ai>

File: ros2/src/openamrobot_description/urdf/robo_urdf.urdf.xacro (robot description, xacro)
@@ -58,9 +58,12 @@
     <collision>
       <!-- Chassis box, CAD Rev B STEP MMP.00.00.00.000: x +-0.390 (panel faces),
-           y +-0.290 (base plate), 0.050 to 0.295 m above the floor (panel bottom to
-           cover top). Was the base_link.STL visual mesh, superseded (#49). -->
-      <origin xyz="0 0 0.0745" rpy="0 0 0"/>
-      <geometry>
-        <box size="0.780 0.580 0.245"/>
+           y +-0.290 (base plate), 0.055 to 0.295 m above the floor (cover top).
+           The bottom sits at 0.055, not the 0.050 panel bottom, so the box clears the
+           caster-wheel collision spheres (top 0.0524 m above the floor) by 2.6 mm;
+           a permanent box/sphere overlap would be a self-collision for MoveIt.
+           Was the base_link.STL visual mesh, superseded (#49). -->
+      <origin xyz="0 0 0.077" rpy="0 0 0"/>
+      <geometry>
+        <box size="0.780 0.580 0.240"/>
       </geometry>
     </collision>

Commit message: description: 2.0 base model, CAD v0.2 chassis with BOM 7.10 components
Replace the May 2026 SolidWorks visual meshes of openamrobot_description.
The chassis comes from the v0.2 full-assembly STEP of openamr-platform-hw
(Rev B panels, 2.0 sensor mounts); release 001 parts in that STEP are
excluded; the 2.0 components of BOM Issue 7.10 are simplified envelopes,
on their sensor, wheel and caster links or as in the CAD.

- tools/cad/step_to_description_meshes.py, cadlib.py and base_mesh_map.yaml
  regenerate the meshes reproducibly (OCP/XCAF, every leaf instance
  classified, envelopes from mapped dimensions, engineering checks)
- meshes/visual: base_chassis, base_covers, base_equipment,
  hub_motor_wheel, caster, lidar, base_camera, ultrasonic, tof, imu
  (2.5 MB in total); meshes/PROVENANCE.yaml records inputs and classes
- URDF: new visuals and materials only; no link, joint, frame, collision
  or inertial change. robot.sdf points at the identical copies in
  meshes/collision
- test_description_meshes.py (14 tests) and a description-tests workflow
- NOTICE.md, STATE.md and the package README updated

Co-Authored-By: Claude Opus 5.5 <noreply@anthropic.com>
Claude-Session: https://claude.ai/code/session_01LwTsQAzAHpEbojLYap63cP
Signed-off-by: Alex Reznichenko <info@botshare.ai>

File: ros2/src/openamrobot_description/urdf/robo_urdf.urdf.xacro (robot description, xacro)
@@ -15,4 +15,24 @@
        in that old origin. They are shifted by z -0.034533 (0.063467 - 0.098) so they
        keep their height above the floor; the meshes themselves are unchanged. -->
+  <!-- Visual materials of the 2.0 base meshes; the colours are listed per mesh in
+       meshes/PROVENANCE.yaml (chassis colours taken from the CAD). -->
+  <material name="chassis_steel">
+    <color rgba="0.352 0.352 0.352 1"/>
+  </material>
+  <material name="chassis_cover">
+    <color rgba="0.352 0.352 0.352 1"/>
+  </material>
+  <material name="equipment_dark">
+    <color rgba="0.2 0.2 0.22 1"/>
+  </material>
+  <material name="hub_motor_dark">
+    <color rgba="0.12 0.12 0.13 1"/>
+  </material>
+  <material name="caster_grey">
+    <color rgba="0.55 0.56 0.58 1"/>
+  </material>
+  <material name="imu_board">
+    <color rgba="0.05 0.12 0.07 1"/>
+  </material>
   <link name="base_footprint"/>
   <!-- base_footprint to base_link: z 0.098 (Alex decision 2026-10-12, STEP MMP.00.00.00.000) -->
@@ -40,19 +60,29 @@
         izz="0.135705995449285" />
     </inertial>
-    <visual>
-      <!-- legacy mesh kept at its floor height: z -0.034533 (Alex decision 2026-10-12);
-           was xyz="0 0 0", superseded by Alex decision 2026-10-12 -->
-      <origin
-        xyz="0 0 -0.034533"
-        rpy="0 0 0" />
-      <geometry>
-        <mesh
-          filename="package://openamrobot_description/meshes/visual/base_link.STL" />
-      </geometry>
-      <material
-        name="">
-        <color
-          rgba="0.792156862745098 0.819607843137255 0.933333333333333 1" />
-      </material>
+    <!-- 2.0 base visual: the chassis from the v0.2 full-assembly STEP (openamr-platform-hw,
+         Rev B panels, 2.0 sensor mounts) and the BOM 7.10 components as envelopes, generated by
+         tools/cad/step_to_description_meshes.py; inputs and parameters in meshes/PROVENANCE.yaml.
+         Was the May 2026 SolidWorks base_link.STL at z -0.034533, superseded. -->
+    <visual>
+      <origin xyz="0 0 0" rpy="0 0 0"/>
+      <geometry>
+        <mesh filename="package://openamrobot_description/meshes/visual/base_chassis.stl"/>
+      </geometry>
+      <material name="chassis_steel"/>
+    </visual>
+    <visual>
+      <origin xyz="0 0 0" rpy="0 0 0"/>
+      <geometry>
+        <mesh filename="package://openamrobot_description/meshes/visual/base_covers.stl"/>
+      </geometry>
+      <material name="chassis_cover"/>
+    </visual>
+    <!-- motor driver, compute, base controller and the battery enclosure (position not decided) -->
+    <visual>
+      <origin xyz="0 0 0" rpy="0 0 0"/>
+      <geometry>
+        <mesh filename="package://openamrobot_description/meshes/visual/base_equipment.stl"/>
+      </geometry>
+      <material name="equipment_dark"/>
     </visual>
     <collision>
@@ -85,17 +115,12 @@
         izz="8.07647021403621E-06" />
     </inertial>
-    <visual>
-      <origin
-        xyz="0 0 0"
-        rpy="0 0 0" />
-      <geometry>
-        <mesh
-          filename="package://openamrobot_description/meshes/visual/fl_caster_link.STL" />
-      </geometry>
-      <material
-        name="">
-        <color
-          rgba="0.792156862745098 0.819607843137255 0.933333333333333 1" />
-      </material>
+    <!-- LPA-VSTH 35K castor envelope (BOM 7.10 MEC-002), wheel included; was the
+         SolidWorks fl_caster_link.STL and fl_wheel_link.STL, superseded -->
+    <visual>
+      <origin xyz="0 0 0" rpy="0 0 0"/>
+      <geometry>
+        <mesh filename="package://openamrobot_description/meshes/visual/caster.stl"/>
+      </geometry>
+      <material name="caster_grey"/>
     </visual>
     <collision>
@@ -140,18 +165,5 @@
         izz="3.74071666197272E-06" />
     </inertial>
-    <visual>
-      <origin
-        xyz="0 0 0"
-        rpy="0 0 0" />
-      <geometry>
-        <mesh
-          filename="package://openamrobot_description/meshes/visual/fl_wheel_link.STL" />
-      </geometry>
-      <material
-        name="">
-        <color
-          rgba="0.792156862745098 0.819607843137255 0.933333333333333 1" />
-      </material>
-    </visual>
+    <!-- no visual: the castor wheel is part of caster.stl on fl_caster_link -->
     <collision>
       <origin xyz="0 0 0" rpy="0 0 0"/>
@@ -191,17 +203,12 @@
         izz="8.07647021403615E-06" />
     </inertial>
-    <visual>
-      <origin
-        xyz="0 0 0"
-        rpy="0 0 0" />
-      <geometry>
-        <mesh
-          filename="package://openamrobot_description/meshes/visual/fr_caster_link.STL" />
-      </geometry>
-      <material
-        name="">
-        <color
-          rgba="0.792156862745098 0.819607843137255 0.933333333333333 1" />
-      </material>
+    <!-- LPA-VSTH 35K castor envelope (BOM 7.10 MEC-002), wheel included; was the
+         SolidWorks fr_caster_link.STL and fr_wheel_link.STL, superseded -->
+    <visual>
+      <origin xyz="0 0 0" rpy="0 0 0"/>
+      <geometry>
+        <mesh filename="package://openamrobot_description/meshes/visual/caster.stl"/>
+      </geometry>
+      <material name="caster_grey"/>
     </visual>
     <collision>
@@ -246,18 +253,5 @@
         izz="3.25059576514846E-06" />
     </inertial>
-    <visual>
-      <origin
-        xyz="0 0 0"
-        rpy="0 0 0" />
-      <geometry>
-        <mesh
-          filename="package://openamrobot_description/meshes/visual/fr_wheel_link.STL" />
-      </geometry>
-      <material
-        name="">
-        <color
-          rgba="0.792156862745098 0.819607843137255 0.933333333333333 1" />
-      </material>
-    </visual>
+    <!-- no visual: the castor wheel is part of caster.stl on fr_caster_link -->
     <collision>
       <origin xyz="0 0 0" rpy="0 0 0"/>
@@ -297,17 +291,12 @@
         izz="8.07647021403621E-06" />
     </inertial>
-    <visual>
-      <origin
-        xyz="0 0 0"
-        rpy="0 0 0" />
-      <geometry>
-        <mesh
-          filename="package://openamrobot_description/meshes/visual/br_caster_link.STL" />
-      </geometry>
-      <material
-        name="">
-        <color
-          rgba="0.792156862745098 0.819607843137255 0.933333333333333 1" />
-      </material>
+    <!-- LPA-VSTH 35K castor envelope (BOM 7.10 MEC-002), wheel included; was the
+         SolidWorks br_caster_link.STL and br_wheel_link.STL, superseded -->
+    <visual>
+      <origin xyz="0 0 0" rpy="0 0 0"/>
+      <geometry>
+        <mesh filename="package://openamrobot_description/meshes/visual/caster.stl"/>
+      </geometry>
+      <material name="caster_grey"/>
     </visual>
     <collision>
@@ -352,18 +341,5 @@
         izz="3.25059576515051E-06" />
     </inertial>
-    <visual>
-      <origin
-        xyz="0 0 0"
-        rpy="0 0 0" />
-      <geometry>
-        <mesh
-          filename="package://openamrobot_description/meshes/visual/br_wheel_link.STL" />
-      </geometry>
-      <material
-        name="">
-        <color
-          rgba="0.792156862745098 0.819607843137255 0.933333333333333 1" />
-      </material>
-    </visual>
+    <!-- no visual: the castor wheel is part of caster.stl on br_caster_link -->
     <collision>
       <origin xyz="0 0 0" rpy="0 0 0"/>
@@ -403,17 +379,12 @@
         izz="8.07647021403621E-06" />
     </inertial>
-    <visual>
-      <origin
-        xyz="0 0 0"
-        rpy="0 0 0" />
-      <geometry>
-        <mesh
-          filename="package://openamrobot_description/meshes/visual/bl_caster_link.STL" />
-      </geometry>
-      <material
-        name="">
-        <color
-          rgba="0.792156862745098 0.819607843137255 0.933333333333333 1" />
-      </material>
+    <!-- LPA-VSTH 35K castor envelope (BOM 7.10 MEC-002), wheel included; was the
+         SolidWorks bl_caster_link.STL and bl_wheel_link.STL, superseded -->
+    <visual>
+      <origin xyz="0 0 0" rpy="0 0 0"/>
+      <geometry>
+        <mesh filename="package://openamrobot_description/meshes/visual/caster.stl"/>
+      </geometry>
+      <material name="caster_grey"/>
     </visual>
     <collision>
@@ -458,18 +429,5 @@
         izz="3.25059576514932E-06" />
     </inertial>
-    <visual>
-      <origin
-        xyz="0 0 0"
-        rpy="0 0 0" />
-      <geometry>
-        <mesh
-          filename="package://openamrobot_description/meshes/visual/bl_wheel_link.STL" />
-      </geometry>
-      <material
-        name="">
-        <color
-          rgba="0.792156862745098 0.819607843137255 0.933333333333333 1" />
-      </material>
-    </visual>
+    <!-- no visual: the castor wheel is part of caster.stl on bl_caster_link -->
     <collision>
       <origin xyz="0 0 0" rpy="0 0 0"/>
@@ -509,17 +467,12 @@
         izz="0.0033973895137008" />
     </inertial>
-    <visual>
-      <origin
-        xyz="0 0 0"
-        rpy="0 0 0" />
-      <geometry>
-        <mesh
-          filename="package://openamrobot_description/meshes/visual/left_wheel_link.STL" />
-      </geometry>
-      <material
-        name="">
-        <color
-          rgba="0.792156862745098 0.819607843137255 0.933333333333333 1" />
-      </material>
+    <!-- ZLLG80ASM250-L-B hub motor wheel envelope, revolved profile from the B2 double-shaft
+         STEP (brake side inboard); was the SolidWorks left_wheel_link.STL, superseded -->
+    <visual>
+      <origin xyz="0 0 0" rpy="0 0 0"/>
+      <geometry>
+        <mesh filename="package://openamrobot_description/meshes/visual/hub_motor_wheel.stl"/>
+      </geometry>
+      <material name="hub_motor_dark"/>
     </visual>
     <collision>
@@ -565,17 +518,12 @@
         izz="0.0033973895137008" />
     </inertial>
-    <visual>
-      <origin
-        xyz="0 0 0"
-        rpy="0 0 0" />
-      <geometry>
-        <mesh
-          filename="package://openamrobot_description/meshes/visual/right_wheel_link.STL" />
-      </geometry>
-      <material
-        name="">
-        <color
-          rgba="0.792156862745098 0.819607843137255 0.933333333333333 1" />
-      </material>
+    <!-- ZLLG80ASM250-L-B hub motor wheel envelope, revolved profile from the B2 double-shaft
+         STEP (brake side inboard, mesh turned by yaw pi); was the SolidWorks right_wheel_link.STL, superseded -->
+    <visual>
+      <origin xyz="0 0 0" rpy="0 0 ${pi}"/>
+      <geometry>
+        <mesh filename="package://openamrobot_description/meshes/visual/hub_motor_wheel.stl"/>
+      </geometry>
+      <material name="hub_motor_dark"/>
     </visual>
     <collision>
@@ -621,15 +569,14 @@
         izz="0.000100924865484583" />
     </inertial>
-    <!-- RPLIDAR S3 body: cylinder 0.0556 m diameter, 0.0413 m high, 0.0277 m below
-         to 0.0136 m above the scan plane (CAD Rev B). Was the A1 lidar_link.STL
-         mesh, superseded (#49). The inertial above is still the A1 one. -->
-    <visual>
-      <origin xyz="0 0 -0.00765" rpy="0 0 0"/>
-      <geometry>
-        <cylinder radius="0.0278" length="0.0413"/>
-      </geometry>
-      <material name="lidar_black">
-        <color rgba="0.1 0.1 0.1 1"/>
-      </material>
+    <!-- RPLIDAR S3 envelope from the STEP instance: body 0.0556 m and head 0.0546 m
+         diameter, 0.0413 m high, base 0.03055 m below the scan plane on the 17.5 mm spacer
+         (NAV-LIDAR stack). Was the cylinder from 0.0277 m below to 0.0136 m above the scan plane
+         (#49), superseded. The collision cylinder and the inertial (still the A1 one) are unchanged. -->
+    <visual>
+      <origin xyz="0 0 0" rpy="0 0 0"/>
+      <geometry>
+        <mesh filename="package://openamrobot_description/meshes/visual/lidar.stl"/>
+      </geometry>
+      <material name="sensor_black"/>
     </visual>
     <collision>

File: ros2/src/openamrobot_description/urdf/sensors.xacro (robot description, xacro)
@@ -18,10 +18,12 @@
     value="${dict(bt05=-0.0873, bt10=-0.1745, bt15=-0.2618)['$(arg base_tilt)']}"/>
   <!-- Origin of the Gemini 336L model in the CAD, front glass, centre of the body.
-       Body 0.029 x 0.124 x 0.029 m behind it. -->
+       Visual: envelope from the STEP instance, body 0.027 x 0.124 x 0.029 m behind the
+       frame and 2.2 mm of glass ahead of it (meshes/PROVENANCE.yaml); was a
+       0.029 x 0.124 x 0.029 m box, superseded. -->
   <link name="base_camera_link">
     <visual>
-      <origin xyz="-0.0124 0 0" rpy="0 0 0"/>
+      <origin xyz="0 0 0" rpy="0 0 0"/>
       <geometry>
-        <box size="0.029 0.124 0.029"/>
+        <mesh filename="package://openamrobot_description/meshes/visual/base_camera.stl"/>
       </geometry>
       <material name="sensor_black"/>
@@ -60,5 +62,15 @@
        Was (0.0544, 0, 0.133) rpy 0 (16 Oct; 177 mm was measured against a
        displaced base plate) and (0.195, 0, -0.044) (Alex decision 2026-10-12). -->
-  <link name="imu_link"/>
+  <!-- Visual: ICM-42688-P package (2.5 x 3.0 x 0.91 mm) on the MIKROE-4237 board,
+       envelope in meshes/visual/imu.stl -->
+  <link name="imu_link">
+    <visual>
+      <origin xyz="0 0 0" rpy="0 0 0"/>
+      <geometry>
+        <mesh filename="package://openamrobot_description/meshes/visual/imu.stl"/>
+      </geometry>
+      <material name="imu_board"/>
+    </visual>
+  </link>
   <joint name="imu_joint" type="fixed">
     <origin xyz="0.0544 0 0.1210" rpy="0 0 ${-pi/2}"/>
@@ -69,10 +81,11 @@
        x along the beam; positive pitch tilts the beam down. -->
   <xacro:macro name="tof_frame" params="name x y z pitch yaw:=0">
-    <!-- TF-Luna body 0.014 x 0.031 x 0.021 m behind the lens face -->
+    <!-- TF-Luna envelope, 0.035 x 0.02125 m, 0.0135 m deep behind the lens face (datasheet
+         A05 and the STEP instance); was a 0.014 x 0.031 x 0.021 m box, superseded -->
     <link name="${name}">
       <visual>
-        <origin xyz="-0.007 0 0" rpy="0 0 0"/>
+        <origin xyz="0 0 0" rpy="0 0 0"/>
         <geometry>
-          <box size="0.014 0.031 0.021"/>
+          <mesh filename="package://openamrobot_description/meshes/visual/tof.stl"/>
         </geometry>
         <material name="sensor_black"/>
@@ -86,10 +99,12 @@
   </xacro:macro>
   <xacro:macro name="ultrasonic_frame" params="name x y z yaw:=0">
-    <!-- MaxSonar WR housing, cylinder 0.031 m diameter, 0.0385 m long behind the face -->
+    <!-- MB7060 -2XX compact housing envelope (datasheet 11838ab): 3/4 inch NPS section
+         0.0262 x 0.0144 m and body 0.0347 x 0.0179 m behind the face, lock nut behind the
+         panel; was a 0.031 m x 0.0385 m cylinder, superseded -->
     <link name="${name}">
       <visual>
-        <origin xyz="-0.01925 0 0" rpy="0 ${pi/2} 0"/>
+        <origin xyz="0 0 0" rpy="0 0 0"/>
         <geometry>
-          <cylinder radius="0.0155" length="0.0385"/>
+          <mesh filename="package://openamrobot_description/meshes/visual/ultrasonic.stl"/>
         </geometry>
         <material name="sensor_black"/>
